Commit message: gazebo

File: urdf/3WD_Omnibot.urdf.xacro (robot description, xacro)
@@ -1,6 +1,9 @@
 <?xml version="1.0"?>
-<robot name="macroed" xmlns:xacro="http://ros.org/wiki/xacro">
+<robot name="omnibot" xmlns:xacro="http://ros.org/wiki/xacro">
+  <xacro:property name="PI" value="3.1415926535897931"/>
+  <xacro:property name="mass" value="1" /> <!-- arbitrary value for mass -->
   <xacro:property name="height" value="0.115" />
-  <xacro:property name="wheeldiam" value="0.04" />
+  <xacro:property name="wheelrad" value="0.05" />
+  <xacro:property name="wheellen" value="0.03" />
   <xacro:property name="R" value="0.15" />
   <xacro:property name="R2" value="0.125" />
@@ -8,13 +11,12 @@
   <xacro:property name="back_wheel_theta" value="${180/180*pi}" />
   <xacro:property name="right_wheel_theta" value="${300/180*pi}" />
-  <material name="dark_grey">
-    <color rgba="0 0 0.8 1"/>
-  </material>
-  <material name="grey">
-    <color rgba="0.1 0.1 0.1 1"/>
-  </material>
-  <material name="yellow">
-    <color rgba="0.8 0.8 0.2 1"/>
-  </material>
+  <xacro:include filename="$(find nexus_base_ros)/urdf/3WD_Omnibot.gazebo" />
+  <xacro:include filename="$(find nexus_base_ros)/urdf/materials.xacro" />
+  <!-- Used for fixing robot to Gazebo 'base_link' -->
+  <link name="footprint"/>
+  <joint name="base_joint" type="fixed">
+    <parent link="footprint"/>
+    <child link="base_link"/>
+  </joint>
   <link name="base_link">
     <visual>
@@ -24,13 +26,22 @@
       <material name="yellow"/>
     </visual>
-    <collision>
-      <geometry>
-        <cylinder radius="${R}" length="${height}"/>
-      </geometry>
-    </collision>
+		<collision>
+			<origin xyz="0 0 ${height/2}" rpy="0 0 0" />
+			<geometry>
+				<cylinder radius="${R}" length="${height}"/>
+			</geometry>
+		</collision>
+		<inertial>
+      <origin xyz="0 0 0" rpy="0 0 0"/>
+      <mass value="${mass}"/>
+      <inertia
+	      ixx="${mass / 12.0 * (3*(R*R) + height*height)}" ixy="0.0" ixz="0.0"
+	      iyy="${mass / 12.0 * (3*(R*R) + height*height)}" iyz="0.0"
+	      izz="${mass / 2.0 * (R*R)}"/>
+    </inertial>
   </link>
 	<link name="left_wheel_link">
 		<visual>
-			<origin  rpy="${pi/2} 0 0" />
+			<origin  rpy="${PI/2} 0 0" />
 			<geometry>
 				<mesh filename="package://nexus_base_ros/meshes/mecanum_wheel.dae"/>
@@ -39,9 +50,17 @@
 		</visual>
 		<collision>
-			<origin xyz="0 0 0" rpy="${pi/2} 0 0" />
+			<origin xyz="0 0 0" rpy="${PI/2} 0 0" />
 			<geometry>
-				<cylinder radius="${wheeldiam/2}" length="0.1"/>
+				<cylinder radius="${wheelrad}" length="${wheellen}"/>
 			</geometry>
 		</collision>
+		<inertial>
+      <origin xyz="0 0 ${wheellen/2}" rpy="0 0 0"/>
+      <mass value="${mass}"/>
+      <inertia
+	      ixx="${mass / 12.0 * (3*(wheelrad*wheelrad) + wheellen*wheellen)}" ixy="0.0" ixz="0.0"
+	      iyy="${mass / 12.0 * (3*(wheelrad*wheelrad) + wheellen*wheellen)}" iyz="0.0"
+	      izz="${mass / 2.0 * (wheelrad*wheelrad)}"/>
+    </inertial>
 	</link>
 	<joint name="left_wheel_joint" type="continuous">
@@ -49,9 +68,10 @@
 		<parent link="base_link"/>
 		<child link="left_wheel_link"/>
-		<origin xyz="${R2*cos(left_wheel_theta)} ${R2*sin(left_wheel_theta)} 0" rpy="0 0 ${left_wheel_theta-pi/2}"/>
+		<origin xyz="${R2*cos(left_wheel_theta)} ${R2*sin(left_wheel_theta)} 0" rpy="0 0 ${left_wheel_theta+PI/2}"/>
+		<dynamics damping="0.7"/>
 	</joint>
 	<link name="back_wheel_link">
 		<visual>
-			<origin  rpy="${back_wheel_theta+pi/2} 0 0" />
+			<origin  rpy="${back_wheel_theta+PI/2} 0 0" />
 			<geometry>
 				<mesh filename="package://nexus_base_ros/meshes/mecanum_wheel.dae"/>
@@ -60,9 +80,17 @@
 		</visual>
 		<collision>
-		<origin xyz="0 0 0" rpy="${pi/2} 0 0" />
+			<origin xyz="0 0 0" rpy="${PI/2} 0 0" />
 			<geometry>
-				<cylinder radius="${wheeldiam/2}" length="0.1"/>
+				<cylinder radius="${wheelrad}" length="${wheellen}"/>
 			</geometry>
 		</collision>
+		<inertial>
+      <origin xyz="0 0 ${wheellen/2}" rpy="0 0 0"/>
+      <mass value="${mass}"/>
+      <inertia
+	      ixx="${mass / 12.0 * (3*(wheelrad*wheelrad) + wheellen*wheellen)}" ixy="0.0" ixz="0.0"
+	      iyy="${mass / 12.0 * (3*(wheelrad*wheelrad) + wheellen*wheellen)}" iyz="0.0"
+	      izz="${mass / 2.0 * (wheelrad*wheelrad)}"/>
+    </inertial>
 	</link>
 	<joint name="back_wheel_joint" type="continuous">
@@ -70,9 +98,10 @@
 		<parent link="base_link"/>
 		<child link="back_wheel_link"/>
-		<origin xyz="${R2*cos(back_wheel_theta)} ${R2*sin(back_wheel_theta)} 0" rpy="0 0 ${back_wheel_theta-pi/2}"/>
+		<origin xyz="${R2*cos(back_wheel_theta)} ${R2*sin(back_wheel_theta)} 0" rpy="0 0 ${back_wheel_theta-PI/2}"/>
+		<dynamics damping="0.7"/>
 	</joint>
 	<link name="right_wheel_link">
 		<visual>
-		<origin  rpy="${pi/2} 0 0" />
+		<origin  rpy="${PI/2} 0 0" />
 		<geometry>
 			<mesh filename="package://nexus_base_ros/meshes/mecanum_wheel.dae"/>
@@ -81,9 +110,17 @@
 		</visual>
 		<collision>
-			<origin  rpy="${pi/2} 0 0" />
+			<origin xyz="0 0 0" rpy="${PI/2} 0 0" />
 			<geometry>
-				<cylinder radius="${wheeldiam/2}" length="0.1"/>
+				<cylinder radius="${wheelrad}" length="${wheellen}"/>
 			</geometry>
 		</collision>
+		<inertial>
+      <origin xyz="0 0 ${wheellen/2}" rpy="0 0 0"/>
+      <mass value="${mass}"/>
+      <inertia
+	      ixx="${mass / 12.0 * (3*(wheelrad*wheelrad) + wheellen*wheellen)}" ixy="0.0" ixz="0.0"
+	      iyy="${mass / 12.0 * (3*(wheelrad*wheelrad) + wheellen*wheellen)}" iyz="0.0"
+	      izz="${mass / 2.0 * (wheelrad*wheelrad)}"/>
+    </inertial>
 	</link>
 	<joint name="right_wheel_joint" type="continuous">
@@ -91,5 +128,6 @@
 		<parent link="base_link"/>
 		<child link="right_wheel_link"/>
-		<origin xyz="${R2*cos(right_wheel_theta)} ${R2*sin(right_wheel_theta)} 0" rpy="0 0 ${right_wheel_theta-pi/2}"/>
+		<origin xyz="${R2*cos(right_wheel_theta)} ${R2*sin(right_wheel_theta)} 0" rpy="0 0 ${right_wheel_theta+PI/2}"/>
+		<dynamics damping="0.7"/>
 	</joint>
 	<link name="lidar_link">
@@ -107,3 +145,33 @@
 		<origin xyz="0.095 0 0.115" rpy="0 0 0" />
 	</joint>
+  <transmission name="left_wheel_tran">
+    <type>transmission_interface/SimpleTransmission</type>
+    <joint name="left_wheel_joint">
+      <hardwareInterface>hardware_interface/EffortJointInterface</hardwareInterface>
+    </joint>
+    <actuator name="left_wheel_motor">
+      <hardwareInterface>hardware_interface/EffortJointInterface</hardwareInterface>
+      <mechanicalReduction>1</mechanicalReduction>
+    </actuator>
+  </transmission>
+  <transmission name="back_wheel_tran">
+    <type>transmission_interface/SimpleTransmission</type>
+    <joint name="back_wheel_joint">
+      <hardwareInterface>hardware_interface/EffortJointInterface</hardwareInterface>
+    </joint>
+    <actuator name="back_wheel_motor">
+      <hardwareInterface>hardware_interface/EffortJointInterface</hardwareInterface>
+      <mechanicalReduction>1</mechanicalReduction>
+    </actuator>
+  </transmission>
+  <transmission name="right_wheel_tran">
+    <type>transmission_interface/SimpleTransmission</type>
+    <joint name="right_wheel_joint">
+      <hardwareInterface>hardware_interface/EffortJointInterface</hardwareInterface>
+    </joint>
+    <actuator name="right_wheel_motor">
+      <hardwareInterface>hardware_interface/EffortJointInterface</hardwareInterface>
+      <mechanicalReduction>1</mechanicalReduction>
+    </actuator>
+  </transmission>
 </robot>

Commit message: updated readme

File: urdf/3WD_Omnibot.urdf.xacro (robot description, xacro)
@@ -145,4 +145,10 @@
 		<origin xyz="0.095 0 0.115" rpy="0 0 0" />
 	</joint>
+	<link name="laser_frame"/>
+	<joint name="laser_lidar_joint" type="fixed">
+		<parent link="lidar_link"/>
+		<child link="laser_frame"/>
+		<origin xyz="0 0 0.06" rpy="0 0 0" />
+	</joint>
   <transmission name="left_wheel_tran">
     <type>transmission_interface/SimpleTransmission</type>
